File: arduino-ir-relay.sch (KiCad schematic (older format))
At the start: 16 parts, among them J0 Screw_Terminal_01x02, J1 Conn_02x03_Row_Letter_First, J2 Conn_02x03_Row_Letter_First, J3 Conn_02x03_Row_Letter_First, J4 Conn_02x03_Row_Letter_First

Commit message: Updated for Kicad 5
Parts:
- removed ATMEGA1: ATMEGA328P-PU, Housings_DIP:DIP-28_W7.62mm_Socket, symbol ATMEGA328P-PU
- added ATMEGA1: ATmega328P-PU, Package_DIP:DIP-28_W7.62mm, symbol MCU_Microchip_ATmega:ATmega328P-PU
- C1, C2, C3, C4: footprint Capacitors_THT:C_Disc_D3.0mm_W1.6mm_P2.50mm -> Capacitor_THT:C_Disc_D3.0mm_W1.6mm_P2.50mm; symbol C -> Device:C
- CLK1: footprint Crystals:Crystal_HC49-U_Vertical -> Crystal:Crystal_HC49-U_Vertical; symbol Crystal -> Device:Crystal
- D1: footprint LEDs:LED_D5.0mm -> LED_THT:LED_D5.0mm; symbol LED -> Device:LED
- IR1: footprint Opto-Devices:IRReceiver_Vishay_MOLD-3pin -> OptoDevice:Vishay_MOLD-3Pin; symbol TSOP343xx -> Interface_Optical:TSOP343xx
- J0: symbol Screw_Terminal_01x02 -> Connector:Screw_Terminal_01x02
- J1, J2, J3, J4: symbol Conn_02x03_Row_Letter_First -> Connector_Generic:Conn_02x03_Row_Letter_First
- R1, R2: footprint Resistors_THT:R_Axial_DIN0204_L3.6mm_D1.6mm_P5.08mm_Horizontal -> Resistor_THT:R_Axial_DIN0204_L3.6mm_D1.6mm_P5.08mm_Horizontal; symbol R -> Device:R
- VREF1: footprint TO_SOT_Packages_THT:TO-220-3_Vertical -> Package_TO_SOT_THT:TO-220-3_Vertical; symbol L7805 -> Regulator_Linear:L7805
Connections:
- net 5V: now also ATMEGA1.20 (AVCC), ATMEGA1.21 (AREF), ATMEGA1.7 (VCC)
- net GNDREF: now also ATMEGA1.22 (GND), ATMEGA1.8 (GND)
- net S1: now also ATMEGA1.5 (PD3)
- net S2: now also ATMEGA1.6 (PD4)
- net S3: now also ATMEGA1.11 (PD5)
- net S4: now also ATMEGA1.12 (PD6)
- net S5: now also ATMEGA1.13 (PD7)
- net S6: now also ATMEGA1.14 (PB0)
- net S7: now also ATMEGA1.15 (PB1)
- net S8: now also ATMEGA1.16 (PB2)
- net at R2.2: now also ATMEGA1.1 (~RESET~/PC6)
- net at C4.1, CLK1.1: now also ATMEGA1.10 (XTAL2/PB7)
- net at IR1.1 (OUT): now also ATMEGA1.4 (PD2)
- net at C3.1, CLK1.2: now also ATMEGA1.9 (XTAL1/PB6)
Other:
- moved on the sheet: C1, C2, IR1, J0, R1, R2, VREF1
